File: Final Project/PCB Design/test/test.kicad_pcb (KiCad board)
At the start: 4 copper layers, 25 parts

Commit message: Edited pcb
Parts:
- removed REF**: LED_GND, Connector_PinSocket_2.54mm:PinSocket_1x04_P2.54mm_Vertical
- removed REF**: Motor_In, Connector_PinSocket_2.54mm:PinSocket_1x04_P2.54mm_Vertical
- removed REF**: PSoC_BTN_OUT, Connector_PinSocket_2.54mm:PinSocket_1x01_P2.54mm_Vertical
- removed REF** (x6): 470, Resistor_THT:R_Axial_DIN0207_L6.3mm_D2.5mm_P10.16mm_Horizontal
- removed REF**: DIP-16_W7.62mm, Package_DIP:DIP-16_W7.62mm
- removed REF**: SPEAKER_GPIO, Connector_PinSocket_2.54mm:PinSocket_1x01_P2.54mm_Vertical
- removed REF** (x2): CP_Radial_D10.0mm_P7.50mm, Capacitor_THT:CP_Radial_D10.0mm_P7.50mm
- removed REF**: SPEAKER_1, Connector_PinSocket_2.54mm:PinSocket_1x02_P2.54mm_Vertical
- removed REF**: SPEAKER_2, Connector_PinSocket_2.54mm:PinSocket_1x02_P2.54mm_Vertical
- removed REF** (x2): PN2222A, Connector_PinSocket_2.54mm:PinSocket_1x03_P2.54mm_Vertical
- removed REF**: 13.5V Connector, Connector_PinSocket_2.54mm:PinSocket_1x02_P2.54mm_Vertical
- removed REF**: LED_IN, Connector_PinSocket_2.54mm:PinSocket_1x04_P2.54mm_Vertical
- removed REF**: LED_OUT, Connector_PinSocket_2.54mm:PinSocket_1x04_P2.54mm_Vertical
- removed REF**: 5V Connector, Connector_PinSocket_2.54mm:PinSocket_1x02_P2.54mm_Vertical
- removed REF** (x2): 1000, Resistor_THT:R_Axial_DIN0207_L6.3mm_D2.5mm_P10.16mm_Horizontal
- removed REF**: Button, Connector_PinSocket_2.54mm:PinSocket_1x02_P2.54mm_Vertical
- removed REF**: Motor_Out, Connector_PinSocket_2.54mm:PinSocket_1x04_P2.54mm_Vertical
- added C1: 10u, Capacitor_THT:CP_Radial_D10.0mm_P7.50mm, F.Cu at (141.2, 83.8)
- added C2: 10u, Capacitor_THT:CP_Radial_D10.0mm_P7.50mm, F.Cu at (141.2, 96.5)
- added G***: LOGO, Graphics:cat, B.Cu at (116.8, 71.1)
- added J1: MOTOR_INPUT, Connector_PinSocket_2.54mm:PinSocket_1x04_P2.54mm_Vertical, F.Cu at (73.7, 45.7)
- added J10: LED_GND, Connector_PinSocket_2.54mm:PinSocket_1x04_P2.54mm_Vertical, F.Cu at (155.0, 81.3)
- added J11: PSoC_I2C_BUS, Connector_PinHeader_2.54mm:PinHeader_1x02_P2.54mm_Vertical, F.Cu at (129.5, 45.7)
- added J12: 13.5V, Connector_PinHeader_2.54mm:PinHeader_1x02_P2.54mm_Vertical, F.Cu at (73.7, 53.3)
- added J13: RTC_I2C, Connector_PinHeader_2.54mm:PinHeader_1x06_P2.54mm_Vertical, F.Cu at (160.0, 45.7)
- added J14: PSoC_RTC_INT_COT_IN, Connector_PinHeader_2.54mm:PinHeader_1x02_P2.54mm_Vertical, F.Cu at (119.4, 45.7)
- added J15: LED_IN, Connector_PinHeader_2.54mm:PinHeader_1x04_P2.54mm_Vertical, F.Cu at (73.7, 73.7)
- added J2: BTN, Connector_PinHeader_2.54mm:PinHeader_1x02_P2.54mm_Vertical, F.Cu at (149.9, 45.7)
- added J3: SPEAKER_IN_1, Connector_PinHeader_2.54mm:PinHeader_1x02_P2.54mm_Vertical, F.Cu at (154.9, 96.5)
- added J35: Speaker_GPIO, Connector_PinHeader_2.54mm:PinHeader_1x01_P2.54mm_Vertical, F.Cu at (111.8, 45.7)
- added J4: SPEAKER_IN_2, Connector_PinHeader_2.54mm:PinHeader_1x02_P2.54mm_Vertical, F.Cu at (160.0, 96.5)
- added J42: PSoC_BTN_OUT, Connector_PinHeader_2.54mm:PinHeader_1x01_P2.54mm_Vertical, F.Cu at (137.2, 45.7)
- added J43: LCD_I2C, Connector_PinSocket_2.54mm:PinSocket_1x04_P2.54mm_Vertical, F.Cu at (160.0, 64.8)
- added J5: 5V, Connector_PinHeader_2.54mm:PinHeader_1x02_P2.54mm_Vertical, F.Cu at (73.7, 63.5)
- added J9: LED_OUT, Connector_PinSocket_2.54mm:PinSocket_1x04_P2.54mm_Vertical, F.Cu at (160.0, 81.3)
- added M1: Stepper_Motor_bipolar, Connector_PinSocket_2.54mm:PinSocket_1x04_P2.54mm_Vertical, F.Cu at (88.9, 45.7)
- added Q1: PN2222A, Connector_PinHeader_2.54mm:PinHeader_1x03_P2.54mm_Vertical, F.Cu at (134.6, 94.0)
- added Q2: PN2222A, Connector_PinHeader_2.54mm:PinHeader_1x03_P2.54mm_Vertical, F.Cu at (134.6, 81.3)
- added R1: 470, Resistor_THT:R_Axial_DIN0411_L9.9mm_D3.6mm_P12.70mm_Horizontal, F.Cu at (99.1, 85.1)
- added R2: 470, Resistor_THT:R_Axial_DIN0411_L9.9mm_D3.6mm_P12.70mm_Horizontal, F.Cu at (94.0, 85.1)
- added R3: 470, Resistor_THT:R_Axial_DIN0411_L9.9mm_D3.6mm_P12.70mm_Horizontal, F.Cu at (88.9, 85.1)
- added R4: 470, Resistor_THT:R_Axial_DIN0411_L9.9mm_D3.6mm_P12.70mm_Horizontal, F.Cu at (83.8, 85.1)
- added R5: 1000, Resistor_THT:R_Axial_DIN0411_L9.9mm_D3.6mm_P12.70mm_Horizontal, F.Cu at (109.2, 85.1)
- added R6: 1000, Resistor_THT:R_Axial_DIN0411_L9.9mm_D3.6mm_P12.70mm_Horizontal, F.Cu at (119.4, 85.1)
- added R7: 470, Resistor_THT:R_Axial_DIN0411_L9.9mm_D3.6mm_P12.70mm_Horizontal, F.Cu at (114.3, 97.8)
- added R8: 470, Resistor_THT:R_Axial_DIN0411_L9.9mm_D3.6mm_P12.70mm_Horizontal, F.Cu at (124.5, 97.8)
- added U1: L293D, Package_DIP:DIP-16_W7.62mm, F.Cu at (85.1, 54.6)
Routing:
- net (no net): track 879.7 -> 0.00 mm
- net +5V: track 0.00 -> 153.8 mm
- net Net-(J9-Pin_1): track 0.00 -> 83.9 mm
- net Net-(J9-Pin_2): track 0.00 -> 76.9 mm
- net Net-(J9-Pin_3): track 0.00 -> 70.8 mm
- net Net-(J9-Pin_4): track 0.00 -> 64.6 mm
- net Net-(J35-Pin_1): track 0.00 -> 56.8 mm
- net Net-(U1-2Y): track 0.00 -> 53.8 mm
- net Net-(J11-Pin_1): track 0.00 -> 52.9 mm
- net Net-(U1-1Y): track 0.00 -> 47.9 mm
- net Net-(J11-Pin_2): track 0.00 -> 45.8 mm
- net Net-(J13-Pin_2): track 0.00 -> 41.7 mm
- net Net-(J13-Pin_1): track 0.00 -> 40.2 mm
- net Net-(J1-Pin_2): track 0.00 -> 34.5 mm
- net Net-(J1-Pin_3): track 0.00 -> 33.0 mm
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- added copper zone on In1.Cu, net GND
- added copper zone on In2.Cu, net VCC
Other:
- board outline added: 96.5 x 63.5 mm

Commit message: final 3D model design and PCB design
Parts:
- added C3: 100n, Capacitor_THT:C_Disc_D7.5mm_W5.0mm_P5.00mm, F.Cu at (116.8, 71.2)
- added C4: 100n, Capacitor_THT:C_Disc_D7.5mm_W5.0mm_P5.00mm, F.Cu at (124.5, 76.2)
- added J6: ENC_OUT, Connector_PinHeader_2.54mm:PinHeader_1x03_P2.54mm_Vertical, F.Cu at (154.9, 63.5)
- added J7: ENC_IN, Connector_PinHeader_2.54mm:PinHeader_1x02_P2.54mm_Vertical, F.Cu at (142.2, 45.7)
- added R10: 1000, Resistor_THT:R_Axial_DIN0411_L9.9mm_D3.6mm_P12.70mm_Horizontal, F.Cu at (149.9, 76.2)
- added R9: 1000, Resistor_THT:R_Axial_DIN0411_L9.9mm_D3.6mm_P12.70mm_Horizontal, F.Cu at (133.3, 71.1)
Routing:
- net Net-(J6-Pin_1): track 0.00 -> 71.1 mm
- net Net-(J6-Pin_3): track 0.00 -> 60.3 mm
- net +5V: track 153.8 -> 162.3 mm

Commit message: final pcb design?
Parts:
- added C5: 1uF, Capacitor_THT:C_Disc_D8.0mm_W5.0mm_P5.00mm, F.Cu at (81.0, 68.7)
- added C6: .1uF, Capacitor_THT:C_Disc_D8.0mm_W5.0mm_P5.00mm, F.Cu at (96.8, 59.6)
Routing:
- net +5V: track 162.3 -> 7.62 mm
- net Net-(U1-2Y): track 53.8 -> 28.4 mm
- net Net-(U1-1Y): track 47.9 -> 23.5 mm, vias 0 -> 1
- net Net-(J1-Pin_2): track 34.5 -> 37.4 mm
- net Net-(M1--): track 27.9 -> 25.5 mm
- net Net-(U1-4Y): track 14.5 -> 16.6 mm
- net Net-(J15-Pin_1): track 30.1 -> 30.9 mm
- net GND: vias 0 -> 146
- added copper zone on In2.Cu, net +5V
- added copper zone on F.Cu, net GND

Commit message: add lab 6
Routing:
- net Net-(J1-Pin_2): track 37.4 -> 37.9 mm
- net GND: vias 146 -> 90

Commit message: added lab 6
Parts:
- moved C3 0.08 mm to (116.8, 71.1)
Routing:
- net GND: vias 90 -> 62
